File: cinco-cinco/cinco-cinco.kicad_pcb (KiCad board)
At the start: 2 copper layers, 98.1 x 68.1 mm, 12 parts, among them J1 Conn_01x04_Socket, SW1 SW_Push, SW2 SW_Push, SW3 SW_Push, SW4 SW_Push, SW5 SW_Push, U1 MCP23008-xSS

Commit message: so much new schtuff.
Other:
- board text added: "2025-05-22"
- board text added: "cinco cinco"
